Commit message: Change the inerital properties of the cobot

File: agv/agv_description/urdf/agv.urdf.xacro (robot description, xacro)
@@ -28,5 +28,6 @@
 	<!-- IMU Plugin-->
 	<xacro:agv_imu />
-	<xacro:include filename="$(find ur5_cobot)/ur_description/urdf/ur5_robot.urdf.xacro"/>
+	<xacro:include filename="$(find ur5_cobot)/ur_description/urdf/ur5_joint_limited_robot.urdf.xacro"/>
+	<!-- <link name="dummy" /> -->
 	<joint name="base_arm_joint" type="fixed">
 		<parent link="base_link" />

File: agv/agv_description/urdf/agv_base.urdf.xacro (robot description, xacro)
@@ -17,5 +17,6 @@
         </geometry>
       </collision>
-      <xacro:box_inertial x="1.02605" y="0.728"  z="0.3" mass="1.0" />
+      <!-- <xacro:box_inertial x="10.2605" y="7.28"  z="3.0" mass="10.0" /> -->
+      <xacro:box_inertial x="51.3025" y="36.4"  z="15.0" mass="50.0" />
     </link>
     <gazebo reference="base_link">

File: agv/agv_description/urdf/agv_caster.urdf.xacro (robot description, xacro)
@@ -16,5 +16,5 @@
         </geometry>
       </collision>
-      <xacro:cylinder_inertial radius="0.005" length="0.07" mass="0.1" />
+      <xacro:cylinder_inertial radius="0.005" length="0.07" mass="0.5" />
     </link>
     <joint name="caster_${side}_joint" type="continuous">

File: agv/agv_description/urdf/agv_wheel.urdf.xacro (robot description, xacro)
@@ -15,5 +15,5 @@
         </geometry>
       </collision>
-      <xacro:cylinder_inertial radius="0.15" length="0.02" mass="0.1"/>
+      <xacro:cylinder_inertial radius="0.15" length="0.02" mass="0.5"/>
     </link>
     <joint name="wheel_${side}_base" type="continuous">

File: ur_cobot/ur5_cobot/ur_description/urdf/ur.gazebo.xacro (robot description, xacro)
@@ -2,4 +2,7 @@
 <robot xmlns:xacro="http://wiki.ros.org/xacro">
   <xacro:macro name="ur_arm_gazebo" params="prefix">
+    <gazebo reference="${prefix}cobot_base_link">
+      <selfCollide>true</selfCollide>
+    </gazebo>
     <gazebo reference="${prefix}shoulder_link">
       <selfCollide>true</selfCollide>

File: ur_cobot/ur5_cobot/ur_description/urdf/ur5.urdf.xacro (robot description, xacro)
@@ -4,5 +4,5 @@
   <xacro:include filename="$(find ur5_cobot)/ur_description/urdf/ur.gazebo.xacro" />
   <xacro:include filename="$(find ur5_cobot)/ur_description/urdf/kinect.urdf.xacro"/>
-  <xacro:macro name="cylinder_inertial" params="radius length mass *origin">
+  <!-- <xacro:macro name="cylinder_inertial" params="radius length mass *origin">
     <inertial>
       <mass value="${mass}" />
@@ -11,4 +11,13 @@
         iyy="${0.0833333 * mass * (3 * radius * radius + length * length)}" iyz="0.0"
         izz="${0.5 * mass * radius * radius}" />
+    </inertial>
+  </xacro:macro> -->
+  <xacro:macro name="cylinder_inertial" params="radius length mass *origin">
+    <inertial>
+      <mass value="${mass}" />
+      <xacro:insert_block name="origin" />
+      <inertia ixx="0.002" ixy="0.0" ixz="0.0"
+        iyy="0.02" iyz="0.0"
+        izz="0.002" />
     </inertial>
   </xacro:macro>
@@ -105,16 +114,16 @@
       <axis xyz="0 0 1" />
       <xacro:unless value="${joint_limited}">
-        <limit lower="${-2.0 * pi}" upper="${2.0 * pi}" effort="300.0" velocity="3.15"/>
-        <xacro:if value="${safety_limits}">
-          <safety_controller soft_lower_limit="${-2.0 * pi + safety_pos_margin}" soft_upper_limit="${2.0 * pi - safety_pos_margin}" k_position="${safety_k_position}" k_velocity="0.0"/>
-        </xacro:if>
-      </xacro:unless>
-      <xacro:if value="${joint_limited}">
-        <limit lower="${shoulder_pan_lower_limit}" upper="${shoulder_pan_upper_limit}" effort="300.0" velocity="3.15"/>
+        <limit lower="${-2.0 * pi}" upper="${2.0 * pi}" effort="150.0" velocity="3.15"/>
+        <xacro:if value="${safety_limits}">
+          <safety_controller soft_lower_limit="${-2.0 * pi + safety_pos_margin}" soft_upper_limit="${2.0 * pi - safety_pos_margin}" k_position="${safety_k_position}" k_velocity="0.0"/>
+        </xacro:if>
+      </xacro:unless>
+      <xacro:if value="${joint_limited}">
+        <limit lower="${shoulder_pan_lower_limit}" upper="${shoulder_pan_upper_limit}" effort="150.0" velocity="3.15"/>
         <xacro:if value="${safety_limits}">
           <safety_controller soft_lower_limit="${shoulder_pan_lower_limit + safety_pos_margin}" soft_upper_limit="${shoulder_pan_upper_limit - safety_pos_margin}" k_position="${safety_k_position}" k_velocity="0.0"/>
         </xacro:if>
       </xacro:if>
-      <dynamics damping="0.0" friction="0.0"/>
+      <dynamics damping="0.5" friction="0.0"/>
     </joint>
     <link name="${prefix}shoulder_link">
@@ -142,16 +151,16 @@
       <axis xyz="0 1 0" />
       <xacro:unless value="${joint_limited}">
-        <limit lower="${-2.0 * pi}" upper="${2.0 * pi}" effort="300.0" velocity="3.15"/>
-        <xacro:if value="${safety_limits}">
-          <safety_controller soft_lower_limit="${-2.0 * pi + safety_pos_margin}" soft_upper_limit="${2.0 * pi - safety_pos_margin}" k_position="${safety_k_position}" k_velocity="0.0"/>
-        </xacro:if>
-      </xacro:unless>
-      <xacro:if value="${joint_limited}">
-        <limit lower="${shoulder_lift_lower_limit}" upper="${shoulder_lift_upper_limit}" effort="300.0" velocity="3.15"/>
+        <limit lower="${-2.0 * pi}" upper="${2.0 * pi}" effort="150.0" velocity="3.15"/>
+        <xacro:if value="${safety_limits}">
+          <safety_controller soft_lower_limit="${-2.0 * pi + safety_pos_margin}" soft_upper_limit="${2.0 * pi - safety_pos_margin}" k_position="${safety_k_position}" k_velocity="0.0"/>
+        </xacro:if>
+      </xacro:unless>
+      <xacro:if value="${joint_limited}">
+        <limit lower="${shoulder_lift_lower_limit}" upper="${shoulder_lift_upper_limit}" effort="150.0" velocity="3.15"/>
         <xacro:if value="${safety_limits}">
           <safety_controller soft_lower_limit="${shoulder_lift_lower_limit + safety_pos_margin}" soft_upper_limit="${shoulder_lift_upper_limit - safety_pos_margin}" k_position="${safety_k_position}" k_velocity="0.0"/>
         </xacro:if>
       </xacro:if>
-      <dynamics damping="0.0" friction="0.0"/>
+      <dynamics damping="0.5" friction="0.0"/>
     </joint>
     <link name="${prefix}upper_arm_link">
@@ -179,16 +188,16 @@
       <axis xyz="0 1 0" />
       <xacro:unless value="${joint_limited}">
-        <limit lower="${-pi}" upper="${pi}" effort="300.0" velocity="3.15"/>
-        <xacro:if value="${safety_limits}">
-          <safety_controller soft_lower_limit="${-2.0 * pi + safety_pos_margin}" soft_upper_limit="${2.0 * pi - safety_pos_margin}" k_position="${safety_k_position}" k_velocity="0.0"/>
-        </xacro:if>
-      </xacro:unless>
-      <xacro:if value="${joint_limited}">
-        <limit lower="${elbow_joint_lower_limit}" upper="${elbow_joint_upper_limit}" effort="300.0" velocity="3.15"/>
+        <limit lower="${-pi}" upper="${pi}" effort="150.0" velocity="3.15"/>
+        <xacro:if value="${safety_limits}">
+          <safety_controller soft_lower_limit="${-2.0 * pi + safety_pos_margin}" soft_upper_limit="${2.0 * pi - safety_pos_margin}" k_position="${safety_k_position}" k_velocity="0.0"/>
+        </xacro:if>
+      </xacro:unless>
+      <xacro:if value="${joint_limited}">
+        <limit lower="${elbow_joint_lower_limit}" upper="${elbow_joint_upper_limit}" effort="150.0" velocity="3.15"/>
         <xacro:if value="${safety_limits}">
           <safety_controller soft_lower_limit="${elbow_joint_lower_limit + safety_pos_margin}" soft_upper_limit="${elbow_joint_upper_limit - safety_pos_margin}" k_position="${safety_k_position}" k_velocity="0.0"/>
         </xacro:if>
       </xacro:if>
-      <dynamics damping="0.0" friction="1.0"/>
+      <dynamics damping="0.5" friction="0.0"/>
     </joint>
     <link name="${prefix}forearm_link">
@@ -216,16 +225,16 @@
       <axis xyz="0 1 0" />
       <xacro:unless value="${joint_limited}">
-        <limit lower="${-2.0 * pi}" upper="${2.0 * pi}" effort="100.0" velocity="3.2"/>
-        <xacro:if value="${safety_limits}">
-          <safety_controller soft_lower_limit="${-2.0 * pi + safety_pos_margin}" soft_upper_limit="${2.0 * pi - safety_pos_margin}" k_position="${safety_k_position}" k_velocity="0.0"/>
-        </xacro:if>
-      </xacro:unless>
-      <xacro:if value="${joint_limited}">
-        <limit lower="${wrist_1_lower_limit}" upper="${wrist_1_upper_limit}" effort="100.0" velocity="3.2"/>
+        <limit lower="${-2.0 * pi}" upper="${2.0 * pi}" effort="28.0" velocity="3.2"/>
+        <xacro:if value="${safety_limits}">
+          <safety_controller soft_lower_limit="${-2.0 * pi + safety_pos_margin}" soft_upper_limit="${2.0 * pi - safety_pos_margin}" k_position="${safety_k_position}" k_velocity="0.0"/>
+        </xacro:if>
+      </xacro:unless>
+      <xacro:if value="${joint_limited}">
+        <limit lower="${wrist_1_lower_limit}" upper="${wrist_1_upper_limit}" effort="28.0" velocity="3.2"/>
         <xacro:if value="${safety_limits}">
           <safety_controller soft_lower_limit="${wrist_1_lower_limit + safety_pos_margin}" soft_upper_limit="${wrist_1_upper_limit - safety_pos_margin}" k_position="${safety_k_position}" k_velocity="0.0"/>
         </xacro:if>
       </xacro:if>
-      <dynamics damping="0.0" friction="1.0"/>
+      <dynamics damping="0.5" friction="0.0"/>
     </joint>
     <link name="${prefix}wrist_1_link">
@@ -253,16 +262,16 @@
       <axis xyz="0 0 1" />
       <xacro:unless value="${joint_limited}">
-        <limit lower="${-2.0 * pi}" upper="${2.0 * pi}" effort="100.0" velocity="3.2"/>
-        <xacro:if value="${safety_limits}">
-          <safety_controller soft_lower_limit="${-2.0 * pi + safety_pos_margin}" soft_upper_limit="${2.0 * pi - safety_pos_margin}" k_position="${safety_k_position}" k_velocity="0.0"/>
-        </xacro:if>
-      </xacro:unless>
-      <xacro:if value="${joint_limited}">
-        <limit lower="${wrist_2_lower_limit}" upper="${wrist_2_upper_limit}" effort="100.0" velocity="3.2"/>
+        <limit lower="${-2.0 * pi}" upper="${2.0 * pi}" effort="28.0" velocity="3.2"/>
+        <xacro:if value="${safety_limits}">
+          <safety_controller soft_lower_limit="${-2.0 * pi + safety_pos_margin}" soft_upper_limit="${2.0 * pi - safety_pos_margin}" k_position="${safety_k_position}" k_velocity="0.0"/>
+        </xacro:if>
+      </xacro:unless>
+      <xacro:if value="${joint_limited}">
+        <limit lower="${wrist_2_lower_limit}" upper="${wrist_2_upper_limit}" effort="28.0" velocity="3.2"/>
         <xacro:if value="${safety_limits}">
           <safety_controller soft_lower_limit="${wrist_2_lower_limit + safety_pos_margin}" soft_upper_limit="${wrist_2_upper_limit - safety_pos_margin}" k_position="${safety_k_position}" k_velocity="0.0"/>
         </xacro:if>
       </xacro:if>
-      <dynamics damping="0.0" friction="1.0"/>
+      <dynamics damping="0.5" friction="0.0"/>
     </joint>
     <link name="${prefix}wrist_2_link">
@@ -290,16 +299,16 @@
       <axis xyz="0 1 0" />
       <xacro:unless value="${joint_limited}">
-        <limit lower="${-2.0 * pi}" upper="${2.0 * pi}" effort="100.0" velocity="3.2"/>
-        <xacro:if value="${safety_limits}">
-          <safety_controller soft_lower_limit="${-2.0 * pi + safety_pos_margin}" soft_upper_limit="${2.0 * pi - safety_pos_margin}" k_position="${safety_k_position}" k_velocity="0.0"/>
-        </xacro:if>
-      </xacro:unless>
-      <xacro:if value="${joint_limited}">
-        <limit lower="${wrist_3_lower_limit}" upper="${wrist_3_upper_limit}" effort="100.0" velocity="3.2"/>
+        <limit lower="${-2.0 * pi}" upper="${2.0 * pi}" effort="28.0" velocity="3.2"/>
+        <xacro:if value="${safety_limits}">
+          <safety_controller soft_lower_limit="${-2.0 * pi + safety_pos_margin}" soft_upper_limit="${2.0 * pi - safety_pos_margin}" k_position="${safety_k_position}" k_velocity="0.0"/>
+        </xacro:if>
+      </xacro:unless>
+      <xacro:if value="${joint_limited}">
+        <limit lower="${wrist_3_lower_limit}" upper="${wrist_3_upper_limit}" effort="28.0" velocity="3.2"/>
         <xacro:if value="${safety_limits}">
           <safety_controller soft_lower_limit="${wrist_3_lower_limit + safety_pos_margin}" soft_upper_limit="${wrist_3_upper_limit - safety_pos_margin}" k_position="${safety_k_position}" k_velocity="0.0"/>
         </xacro:if>
       </xacro:if>
-      <dynamics damping="0.0" friction="1.0"/>
+      <dynamics damping="0.5" friction="0.0"/>
     </joint>
     <link name="${prefix}wrist_3_link">
@@ -334,319 +343,4 @@
       </collision>
     </link>
-    <link name="vacuum_gripper">
-      <gravity>0</gravity>
-      <visual>
-        <origin rpy="0 0 0" xyz="0 0 0"/>
-        <geometry>
-          <cylinder radius="0.005" length="0.01"/>
-        </geometry>
-        <material name="transparent">
-          <color rgba="0 0 0 0"/>
-        </material>
-      </visual>
-      <inertial>
-        <origin rpy="0 0 0" xyz="0.000000 0.000000 0.000000"/>
-        <mass value="0.0001"/>
-        <inertia ixx="1e-08" ixy="0" ixz="0" iyy="1e-08" iyz="0" izz="1e-08"/>
-      </inertial>
-    </link>
-    <joint name="gripper_joint" type="fixed">
-      <!-- <axis xyz="1 0 0" /> -->
-      <parent link="ee_link" />
-      <child link="vacuum_gripper" />
-      <origin rpy="0 1.5708 0" xyz="0.01 0.0125 0" />
-      <!-- <limit effort="50" velocity="50" lower="0" upper="0" />
-      <dynamics damping="0.0" friction="10"/> -->
-    </joint>
-  <gazebo>
-      <plugin name="gazebo_ros_vacuum_gripper" filename="libgazebo_ros_vacuum_gripper.so">
-        <robotNamespace>/ur5/vacuum_gripper</robotNamespace>
-        <bodyName>vacuum_gripper</bodyName>
-        <topicName>grasping</topicName>
-	<maxForce>50</maxForce>
-        <maxDistance>0.05</maxDistance>
-        <minDistance>0.01</minDistance>
-      </plugin>
-  </gazebo>
-    <link name="vacuum_gripper1">
-      <gravity>0</gravity>
-      <visual>
-        <origin rpy="0 0 0" xyz="0 0 0"/>
-        <geometry>
-          <cylinder radius="0.005" length="0.01"/>
-        </geometry>
-        <material name="transparent">
-          <color rgba="0 0 0 0"/>
-        </material>
-      </visual>
-      <inertial>
-        <origin rpy="0 0 0" xyz="0.000000 0.000000 0.000000"/>
-        <mass value="0.0001"/>
-        <inertia ixx="1e-08" ixy="0" ixz="0" iyy="1e-08" iyz="0" izz="1e-08"/>
-      </inertial>
-    </link>
-    <joint name="gripper_joint1" type="fixed">
-      <!-- <axis xyz="1 0 0" /> -->
-      <parent link="ee_link" />
-      <child link="vacuum_gripper1" />
-      <origin rpy="0 1.5708 0" xyz="0.01 -0.0125 0" />
-      <!-- <limit effort="50" velocity="50" lower="0" upper="0" /> -->
-      <!-- <dynamics damping="0.0" friction="10"/> -->
-    </joint>
-  <gazebo>
-      <plugin name="gazebo_ros_vacuum_gripper1" filename="libgazebo_ros_vacuum_gripper.so">
-        <robotNamespace>/ur5/vacuum_gripper1</robotNamespace>
-        <bodyName>vacuum_gripper1</bodyName>
-        <topicName>grasping1</topicName>
-	<maxForce>50</maxForce>
-        <maxDistance>0.05</maxDistance>
-        <minDistance>0.01</minDistance>
-      </plugin>
-  </gazebo>
-    <link name="vacuum_gripper2">
-      <gravity>0</gravity>
-      <visual>
-        <origin rpy="0 0 0" xyz="0 0 0"/>
-        <geometry>
-          <cylinder radius="0.005" length="0.01"/>
-        </geometry>
-        <material name="transparent">
-          <color rgba="0 0 0 0"/>
-        </material>
-      </visual>
-      <inertial>
-        <origin rpy="0 0 0" xyz="0.000000 0.000000 0.000000"/>
-        <mass value="0.0001"/>
-        <inertia ixx="1e-08" ixy="0" ixz="0" iyy="1e-08" iyz="0" izz="1e-08"/>
-      </inertial>
-    </link>
-    <joint name="gripper_joint2" type="fixed">
-      <!-- <axis xyz="1 0 0" /> -->
-      <parent link="ee_link" />
-      <child link="vacuum_gripper2" />
-      <origin rpy="0 1.5708 0" xyz="0.01 0 0.0125" />
-      <!-- <limit effort="50" velocity="50" lower="0" upper="0" />
-      <dynamics damping="0.0" friction="10"/> -->
-    </joint>
-  <gazebo>
-      <plugin name="gazebo_ros_vacuum_gripper2" filename="libgazebo_ros_vacuum_gripper.so">
-        <robotNamespace>/ur5/vacuum_gripper2</robotNamespace>
-        <bodyName>vacuum_gripper2</bodyName>
-        <topicName>grasping2</topicName>
-	<maxForce>50</maxForce>
-        <maxDistance>0.05</maxDistance>
-        <minDistance>0.01</minDistance>
-      </plugin>
-  </gazebo>
-    <link name="vacuum_gripper3">
-      <gravity>0</gravity>
-      <visual>
-        <origin rpy="0 0 0" xyz="0 0 0"/>
-        <geometry>
-          <cylinder radius="0.005" length="0.01"/>
-        </geometry>
-        <material name="transparent">
-          <color rgba="0 0 0 0"/>
-        </material>
-      </visual>
-      <inertial>
-        <origin rpy="0 0 0" xyz="0.000000 0.000000 0.000000"/>
-        <mass value="0.0001"/>
-        <inertia ixx="1e-08" ixy="0" ixz="0" iyy="1e-08" iyz="0" izz="1e-08"/>
-      </inertial>
-    </link>
-    <joint name="gripper_joint3" type="fixed">
-      <!-- <axis xyz="1 0 0" /> -->
-      <parent link="ee_link" />
-      <child link="vacuum_gripper3" />
-      <origin rpy="0 1.5708 0" xyz="0.01 0 -0.0125" />
-      <!-- <limit effort="50" velocity="50" lower="0" upper="0" />
-      <dynamics damping="0.0" friction="10"/> -->
-    </joint>
-  <gazebo>
-      <plugin name="gazebo_ros_vacuum_gripper3" filename="libgazebo_ros_vacuum_gripper.so">
-        <robotNamespace>/ur5/vacuum_gripper3</robotNamespace>
-        <bodyName>vacuum_gripper3</bodyName>
-        <topicName>grasping2</topicName>
-	<maxForce>50</maxForce>
-        <maxDistance>0.05</maxDistance>
-        <minDistance>0.01</minDistance>
-      </plugin>
-  </gazebo>
-  <link name="vacuum_gripper4">
-    <gravity>0</gravity>
-    <visual>
-      <origin rpy="0 0 0" xyz="0 0 0"/>
-      <geometry>
-        <cylinder radius="0.005" length="0.01"/>
-      </geometry>
-      <material name="transparent">
-        <color rgba="0 0 0 0"/>
-      </material>
-    </visual>
-    <inertial>
-      <origin rpy="0 0 0" xyz="0.000000 0.000000 0.000000"/>
-      <mass value="0.0001"/>
-      <inertia ixx="1e-08" ixy="0" ixz="0" iyy="1e-08" iyz="0" izz="1e-08"/>
-    </inertial>
-  </link>
-  <joint name="gripper_joint4" type="fixed">
-    <!-- <axis xyz="1 0 0" /> -->
-    <parent link="ee_link" />
-    <child link="vacuum_gripper4" />
-    <origin rpy="0 1.5708 0" xyz="0.01 0 0" />
-    <!-- <limit effort="50" velocity="50" lower="0" upper="0" />
-    <dynamics damping="0.0" friction="10"/> -->
-  </joint>
-  <gazebo>
-    <plugin name="gazebo_ros_vacuum_gripper4" filename="libgazebo_ros_vacuum_gripper.so">
-      <robotNamespace>/ur5/vacuum_gripper4</robotNamespace>
-      <bodyName>vacuum_gripper4</bodyName>
-      <topicName>grasping4</topicName>
-  <maxForce>50</maxForce>
-      <maxDistance>0.05</maxDistance>
-      <minDistance>0.01</minDistance>
-    </plugin>
-  </gazebo>
-  <link name="vacuum_gripper5">
-    <gravity>0</gravity>
-    <visual>
-      <origin rpy="0 0 0" xyz="0 0 0"/>
-      <geometry>
-        <cylinder radius="0.005" length="0.01"/>
-      </geometry>
-      <material name="transparent">
-        <color rgba="0 0 0 0"/>
-      </material>
-    </visual>
-    <inertial>
-      <origin rpy="0 0 0" xyz="0.000000 0.000000 0.000000"/>
-      <mass value="0.0001"/>
-      <inertia ixx="1e-08" ixy="0" ixz="0" iyy="1e-08" iyz="0" izz="1e-08"/>
-    </inertial>
-  </link>
-  <joint name="gripper_joint5" type="fixed">
-    <!-- <axis xyz="1 0 0" /> -->
-    <parent link="ee_link" />
-    <child link="vacuum_gripper5" />
-    <origin rpy="0 1.5708 0" xyz="0.01 0.0125 0.0125" />
-    <!-- <limit effort="50" velocity="50" lower="0" upper="0" />
-    <dynamics damping="0.0" friction="10"/> -->
-  </joint>
-<gazebo>
-    <plugin name="gazebo_ros_vacuum_gripper5" filename="libgazebo_ros_vacuum_gripper.so">
-      <robotNamespace>/ur5/vacuum_gripper5</robotNamespace>
-      <bodyName>vacuum_gripper5</bodyName>
-      <topicName>grasping5</topicName>
-<maxForce>50</maxForce>
-      <maxDistance>0.05</maxDistance>
-      <minDistance>0.01</minDistance>
-    </plugin>
-</gazebo>
-  <link name="vacuum_gripper6">
-    <gravity>0</gravity>
-    <visual>
-      <origin rpy="0 0 0" xyz="0 0 0"/>
-      <geometry>
-        <cylinder radius="0.005" length="0.01"/>
-      </geometry>
-      <material name="transparent">
-        <color rgba="0 0 0 0"/>
-      </material>
-    </visual>
-    <inertial>
-      <origin rpy="0 0 0" xyz="0.000000 0.000000 0.000000"/>
-      <mass value="0.0001"/>
-      <inertia ixx="1e-08" ixy="0" ixz="0" iyy="1e-08" iyz="0" izz="1e-08"/>
-    </inertial>
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
File: ur_cobot/ur5_cobot/ur_description/urdf/ur5_joint_limited_robot.urdf.xacro (robot description, xacro)
@@ -20,5 +20,5 @@
   <joint name="world_joint" type="fixed">
     <parent link="world" />
-    <child link = "base_link" />
+    <child link = "cobot_base_link" />
     <origin xyz="0.0 0.0 0.0" rpy="0.0 0.0 0.0" />
   </joint>
